File: kicad PCBs/receptor-IR/receptor-IR.kicad_pcb (KiCad board)
At the start: 2 copper layers, 60 x 40 mm, 9 parts, among them J1 TB_1X2, J2 Conn_01x04, J3 Conn_01x03, J4 Conn_01x03, SW1 SW_SPDT, U1 nodemcu_ESP32-s

Commit message: actualización 19/09/2022
Parts:
- added H2: Mounting_Hole, EESTN5:hole_3mm, F.Cu at (210.0, 49.0)
- moved J1 4.35 mm to (190.6, 30.6)
- moved J3 3.31 mm to (220.2, 53.3), turned to 180 degrees
- moved J2 2.73 mm to (206.9, 29.4)
- moved J4 2.18 mm to (220.2, 48.9), turned to 180 degrees
- moved U1 2.10 mm to (191.2, 49.1)
- moved H1 0.64 mm to (220.4, 29.5)
Connections:
- J1 pad 1: +BATT -> GND
- J1 pad 2: GND -> +BATT
- SW1 pad 1: VCC -> unconnected-(SW1-Pad1)
- SW1 pad 2: +BATT -> VCC
- SW1 pad 3: unconnected-(SW1-Pad3) -> +BATT
Routing:
- net +BATT: track 27.5 -> 8.23 mm
- net VCC: track 87.2 -> 93.7 mm
- net /TRIGGER: track 11.5 -> 16.6 mm
- net /pin_IR: track 38.2 -> 33.4 mm
- net /ECHO: track 11.5 -> 15.1 mm
