File: kicad PCBs/receptor-IR/receptor-IR.kicad_sch (KiCad schematic)
At the start: 8 parts, among them J1 TB_1X2, J2 Conn_01x04, J3 Conn_01x03, J4 Conn_01x03, SW1 SW_SPDT, U1 nodemcu_ESP32-s

Commit message: actualización 19/09/2022
Connections:
- net +BATT: now also J1.2, SW1.3 (C); no longer J1.1, SW1.2 (B)
- net GND: now also J1.1; no longer J1.2
- net VCC: now also SW1.2 (B); no longer SW1.1 (A)
- no-connect marks 1 -> 0
Other:
- moved on the sheet: SW1
Changed lines of the file:
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@@
   (junction (at 64.77 38.1) (diameter 0) (color 0 0 0 0)
   )
-  (no_connect (at 157.48 57.15))
   (polyline (pts (xy 11.43 92.71) (xy 284.48 92.71))
     (stroke (width 0) (type default) (color 0 0 0 0))
@@
     (stroke (width 0) (type default) (color 0 0 0 0))
   )
-  (wire (pts (xy 161.29 50.8) (xy 161.29 52.07))
-    (stroke (width 0) (type default) (color 0 0 0 0))
-  )
   (wire (pts (xy 34.29 68.58) (xy 26.67 68.58))
     (stroke (width 0) (type default) (color 0 0 0 0))
@@
     (stroke (width 0) (type default) (color 0 0 0 0))
   )
-  (wire (pts (xy 157.48 52.07) (xy 161.29 52.07))
-    (stroke (width 0) (type default) (color 0 0 0 0))
-  )
   (wire (pts (xy 62.23 38.1) (xy 64.77 38.1))
     (stroke (width 0) (type default) (color 0 0 0 0))
   )
+  (wire (pts (xy 161.29 50.8) (xy 161.29 57.15))
+    (stroke (width 0) (type default) (color 0 0 0 0))
+  )
   (wire (pts (xy 31.75 55.88) (xy 31.75 72.39))
     (stroke (width 0) (type default) (color 0 0 0 0))
@@
   )
   (polyline (pts (xy 12.7 11.43) (xy 12.7 92.71))
+    (stroke (width 0) (type default) (color 0 0 0 0))
+  )
+  (wire (pts (xy 157.48 57.15) (xy 161.29 57.15))
     (stroke (width 0) (type default) (color 0 0 0 0))
   )
@@
     (pin "1")
   )
-  (symbol (lib_id "EESTN5:SW_SPDT") (at 152.4 54.61 0) (unit 1)
-    (in_bom yes) (on_board yes) (fields_autoplaced)
-    (property "Reference" "SW1" (id 0) (at 152.4 49.53 0))
-    (property "Value" "SW_SPDT" (id 1) (at 152.4 59.69 0)
-      (effects (font (size 1.27 1.27)) hide)
-    )
-    (property "Footprint" "EESTN5:SW_SPDT_TH_Vertical" (id 2) (at 152.4 54.61 0)
-      (effects (font (size 1.27 1.27)) hide)
-    )
-    (property "Datasheet" "" (id 3) (at 152.4 54.61 0))
+  (symbol (lib_id "EESTN5:SW_SPDT") (at 152.4 57.15 180) (unit 1)
+    (in_bom yes) (on_board yes) (fields_autoplaced)
+    (property "Reference" "SW1" (id 0) (at 152.4 52.07 0))
+    (property "Value" "SW_SPDT" (id 1) (at 152.4 52.07 0)
+      (effects (font (size 1.27 1.27)) hide)
+    )
+    (property "Footprint" "EESTN5:SW_SPDT_TH_Vertical" (id 2) (at 152.4 57.15 0)
+      (effects (font (size 1.27 1.27)) hide)
+    )
+    (property "Datasheet" "" (id 3) (at 152.4 57.15 0))
     (pin "1")
     (pin "2")
@@
     (pin "1")
   )
-  (symbol (lib_id "EESTN5:TB_1X2") (at 120.65 52.07 0) (unit 1)
-    (in_bom yes) (on_board yes) (fields_autoplaced)
-    (property "Reference" "J1" (id 0) (at 121.92 40.64 0)
+  (symbol (lib_id "EESTN5:TB_1X2") (at 120.65 52.07 0) (mirror x) (unit 1)
+    (in_bom yes) (on_board yes) (fields_autoplaced)
+    (property "Reference" "J1" (id 0) (at 116.967 50.8 0)
+      (effects (font (size 1.524 1.524)) (justify right))
+    )
+    (property "Value" "TB_1X2" (id 1) (at 116.967 54.61 0)
+      (effects (font (size 1.524 1.524)) (justify right))
+    )
+    (property "Footprint" "EESTN5:BORNERA2_AZUL" (id 2) (at 119.38 53.34 0)
+      (effects (font (size 1.524 1.524)) hide)
+    )
+    (property "Datasheet" "" (id 3) (at 119.38 53.34 0)
       (effects (font (size 1.524 1.524)))
     )
-    (property "Value" "TB_1X2" (id 1) (at 121.92 44.45 0)
-      (effects (font (size 1.524 1.524)))
-    )
-    (property "Footprint" "EESTN5:BORNERA2_AZUL" (id 2) (at 119.38 50.8 0)
-      (effects (font (size 1.524 1.524)) hide)
-    )
-    (property "Datasheet" "" (id 3) (at 119.38 50.8 0)
-      (effects (font (size 1.524 1.524)))
-    )

Commit message: actualización menor, 21/9/22
Parts:
- J1: value TB_1X2 -> entrada de bateria
- J2: value Conn_01x04 -> ultrasonido
- J3, J4: value Conn_01x03 -> vs1838b
Changed lines of the file:
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@@
   (symbol (lib_id "EESTN5:TB_1X2") (at 120.65 52.07 0) (mirror x) (unit 1)
     (in_bom yes) (on_board yes) (fields_autoplaced)
-    (property "Reference" "J1" (id 0) (at 116.967 50.8 0)
+    (property "Reference" "J1" (id 0) (at 116.84 50.8 0)
       (effects (font (size 1.524 1.524)) (justify right))
     )
-    (property "Value" "TB_1X2" (id 1) (at 116.967 54.61 0)
+    (property "Value" "entrada de bateria" (id 1) (at 116.84 54.61 0)
       (effects (font (size 1.524 1.524)) (justify right))
     )
@@
       (effects (font (size 1.27 1.27)) (justify left))
     )
-    (property "Value" "Conn_01x03" (id 1) (at 243.84 34.2899 0)
+    (property "Value" "vs1838b" (id 1) (at 243.84 34.2899 0)
       (effects (font (size 1.27 1.27)) (justify left))
     )
@@
       (effects (font (size 1.27 1.27)) (justify left))
     )
-    (property "Value" "Conn_01x03" (id 1) (at 245.11 71.1199 0)
+    (property "Value" "vs1838b" (id 1) (at 245.11 71.1199 0)
       (effects (font (size 1.27 1.27)) (justify left))
     )
@@
       (effects (font (size 1.27 1.27)) (justify left))
     )
-    (property "Value" "Conn_01x04" (id 1) (at 213.36 49.5299 0)
+    (property "Value" "ultrasonido" (id 1) (at 213.36 49.5299 0)
       (effects (font (size 1.27 1.27)) (justify left))
     )
@@
     )
     (path "/8684e644-f372-462b-87b1-1463d59cced1"
-      (reference "J1") (unit 1) (value "TB_1X2") (footprint "EESTN5:BORNERA2_AZUL")
+      (reference "J1") (unit 1) (value "entrada de bateria") (footprint "EESTN5:BORNERA2_AZUL")
     )
     (path "/fa106f42-7354-4027-bf0d-3e0c9a9df154"
-      (reference "J2") (unit 1) (value "Conn_01x04") (footprint "EESTN5:pin_strip_4")
+      (reference "J2") (unit 1) (value "ultrasonido") (footprint "EESTN5:pin_strip_4")
     )
     (path "/bba0ae24-fd84-4bda-84d1-2a9ed2df0aa9"
-      (reference "J3") (unit 1) (value "Conn_01x03") (footprint "EESTN5:Pin_Header_3")
+      (reference "J3") (unit 1) (value "vs1838b") (footprint "EESTN5:Pin_Header_3")
     )
     (path "/f620cf38-0ae6-48e7-8bdb-c7d3ba30cbc6"
-      (reference "J4") (unit 1) (value "Conn_01x03") (footprint "EESTN5:Pin_Header_3")
+      (reference "J4") (unit 1) (value "vs1838b") (footprint "EESTN5:Pin_Header_3")
     )
     (path "/3f99edba-c0a0-4b61-b3cf-d92df0ef9810"
