File: kicad PCBs/emisor-IR/emisor-IR.kicad_sch (KiCad schematic)
At the start: 8 parts, among them J1 Conn_01x03, Q1 BC548

Commit message: actualización menor, 21/9/22
Parts:
- D1, D2: value LED -> LED_IR
- J1: value Conn_01x03 -> entrada desde esp32
- R2: value R -> 100
Changed lines of the file:
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@@
   (symbol (lib_id "EESTN5:R") (at 170.18 41.275 0) (unit 1)
     (in_bom yes) (on_board yes) (fields_autoplaced)
-    (property "Reference" "R2" (id 0) (at 172.085 40.0049 0)
+    (property "Reference" "R2" (id 0) (at 171.45 40.0049 0)
       (effects (font (size 1.27 1.27)) (justify left))
     )
-    (property "Value" "R" (id 1) (at 172.085 42.5449 0)
+    (property "Value" "100" (id 1) (at 171.45 42.5449 0)
       (effects (font (size 1.27 1.27)) (justify left))
     )
@@
     (in_bom yes) (on_board yes) (fields_autoplaced)
     (property "Reference" "J1" (id 0) (at 137.795 43.18 0))
-    (property "Value" "Conn_01x03" (id 1) (at 137.795 45.72 0))
+    (property "Value" "entrada desde esp32" (id 1) (at 137.795 45.72 0))
     (property "Footprint" "Connector_JST:JST_EH_B3B-EH-A_1x03_P2.50mm_Vertical" (id 2) (at 137.795 52.705 0)
       (effects (font (size 1.27 1.27)) hide)
@@
   (symbol (lib_id "Device:LED") (at 194.31 52.07 90) (unit 1)
     (in_bom yes) (on_board yes)
-    (property "Reference" "D1" (id 0) (at 190.5 52.07 90)
+    (property "Reference" "D1" (id 0) (at 198.12 52.07 90)
       (effects (font (size 1.27 1.27)) (justify right))
     )
-    (property "Value" "LED" (id 1) (at 189.23 54.61 90)
+    (property "Value" "LED_IR" (id 1) (at 198.12 54.61 90)
       (effects (font (size 1.27 1.27)) (justify right))
     )
@@
       (effects (font (size 1.27 1.27)) (justify right))
     )
-    (property "Value" "LED" (id 1) (at 182.88 54.61 90)
+    (property "Value" "LED_IR" (id 1) (at 180.34 54.61 90)
       (effects (font (size 1.27 1.27)) (justify right))
     )
@@
     )
     (path "/a1338d76-5506-43d2-a656-f06f903e7bdc"
-      (reference "D1") (unit 1) (value "LED") (footprint "EESTN5:led_5mm_clear")
+      (reference "D1") (unit 1) (value "LED_IR") (footprint "EESTN5:led_5mm_clear")
     )
     (path "/a817d8da-b0a5-4a30-8d35-2f1c58073e1f"
-      (reference "D2") (unit 1) (value "LED") (footprint "EESTN5:led_5mm_clear")
+      (reference "D2") (unit 1) (value "LED_IR") (footprint "EESTN5:led_5mm_clear")
     )
     (path "/213e4313-acdd-463d-b0ee-72c417ca3458"
@@
     )
     (path "/59ffd455-e2a3-45a7-94e8-4af0540e6ca3"
-      (reference "J1") (unit 1) (value "Conn_01x03") (footprint "Connector_JST:JST_EH_B3B-EH-A_1x03_P2.50mm_Vertical")
+      (reference "J1") (unit 1) (value "entrada desde esp32") (footprint "Connector_JST:JST_EH_B3B-EH-A_1x03_P2.50mm_Vertical")
     )
     (path "/304facc4-c68d-43c2-8ad8-182f62056569"
@@
     )
     (path "/41bca582-eb59-4799-bbdc-84ce308dfda2"
-      (reference "R2") (unit 1) (value "R") (footprint "EESTN5:RES0.3")
+      (reference "R2") (unit 1) (value "100") (footprint "EESTN5:RES0.3")
     )
   )
