File: kicad PCBs/car-complex/car-complex.kicad_pcb (KiCad board)
At the start: 2 copper layers, 100 x 60 mm, 32 parts, among them J1 led rgb, J2 led rgb, J3 led rgb, J4 Conn_01x05_Male, J5 buzzer, J6 TB_1X2, J7 TB_1X2, J8 TB_1X2, J9 salida emisor, SW1 SW_SPDT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

Commit message: actualización 19/09/2022
Parts:
- removed the hole_2mm at (44.5, 78.2)
- removed the hole_2mm at (93.2, 78.2)
- added C5: 220uf, Capacitor_THT:CP_Radial_D5.0mm_P2.00mm, F.Cu at (105.7, 31.8)
- added hole_2mm: VAL**, EESTN5:hole_2mm, F.Cu at (30.0, 30.0)
- added hole_2mm: VAL**, EESTN5:hole_2mm, F.Cu at (30.0, 80.0)
- added hole_2mm: VAL**, EESTN5:hole_2mm, F.Cu at (120.0, 28.4)
- added hole_2mm: VAL**, EESTN5:hole_2mm, F.Cu at (120.0, 80.0)
- C1: value 220uf -> 10uf; footprint EESTN5:CAP_ELEC_10X8mm -> Capacitor_THT:CP_Radial_D5.0mm_P2.00mm
- C4: footprint EESTN5:CAP_ELEC_10X8mm -> Capacitor_THT:CP_Radial_D5.0mm_P2.00mm
- D2, D3, D4, D5, D6, D7, D8, D9: value DIODE -> 1n4001
- J4: value Conn_01x05_Male -> conector a stepper
- J6: value TB_1X2 -> motor izq
- J7: value TB_1X2 -> motor der
- J8: value TB_1X2 -> bateria
- R1: value R -> 1k
- moved C4 70.2 mm to (36.2, 30.7), turned to 180 degrees
- moved J1 37.2 mm to (51.9, 81.5), turned to 180 degrees
- moved C1 6.64 mm to (36.0, 39.0), turned to 180 degrees
- moved D1 4.22 mm to (43.2, 30.6)
- moved C2 4.06 mm to (34.5, 56.5)
- moved C3 3.93 mm to (39.6, 56.8)
- moved R1 3.65 mm to (51.1, 29.3)
- moved J5 3.47 mm to (93.3, 35.2), turned to 180 degrees
- moved J3 3.18 mm to (54.1, 44.8)
- moved J6 2.97 mm to (99.9, 79.9)
- moved J8 2.80 mm to (39.2, 80.0)
- moved J7 2.53 mm to (111.9, 80.0)
- moved G*** 2.01 mm to (29.5, 45.6)
- moved J2 1.65 mm to (48.8, 44.8)
- moved J4 1.65 mm to (39.6, 66.9)
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- renumbered SW1 to switch1
Connections:
- C1 pad 1: +5V -> VCC
- C4 pad 1: VCC -> +5V
- C4 pad 2: Net-(C4-Pad2) -> GND
- D3 pad 1: Net-(C4-Pad2) -> Net-(D3-Pad1)
- D5 pad 1: Net-(C4-Pad2) -> Net-(D3-Pad1)
- D7 pad 1: Net-(C4-Pad2) -> Net-(D3-Pad1)
- D9 pad 1: Net-(C4-Pad2) -> Net-(D3-Pad1)
- U3 pad 10: /IN2 -> /buzzer
- U3 pad 11: /ENB -> unconnected-(U3-Pad11)
- U3 pad 12: /buzzer -> unconnected-(U3-Pad12)
- U3 pad 24: /Pin_led_3 -> unconnected-(U3-Pad24)
- U3 pad 25: /Pin_led_2 -> unconnected-(U3-Pad25)
- U3 pad 26: /Pin_led_1 -> unconnected-(U3-Pad26)
- U3 pad 27: unconnected-(U3-Pad27) -> /Pin_led_3
- U3 pad 28: unconnected-(U3-Pad28) -> /Pin_led_2
- U3 pad 36: unconnected-(U3-Pad36) -> /Pin_led_1
- U3 pad 4: unconnected-(U3-Pad4) -> /IN4
- U3 pad 5: unconnected-(U3-Pad5) -> /IN3
- U3 pad 6: /IN4 -> /ENA
- U3 pad 7: /IN3 -> /IN1
- U3 pad 8: /ENA -> /IN2
- U3 pad 9: /IN1 -> /ENB
Routing:
- net Net-(C4-Pad2): track 89.2 -> 0.00 mm
- net Net-(D3-Pad1): track 0.00 -> 81.7 mm
- net +5V: track 132.3 -> 154.1 mm
- net /Pin_led_1: track 28.2 -> 11.7 mm
- net /pin_IR: track 19.1 -> 7.84 mm
- net /IN4: track 26.8 -> 37.2 mm
- net /buzzer: track 12.9 -> 23.2 mm
- net /Pin_led_3: track 6.05 -> 15.1 mm
- net /IN3: track 23.1 -> 31.9 mm
- net /ENB: track 28.9 -> 36.8 mm
- net /IN1: track 18.3 -> 26.1 mm
- net /IN2: track 23.8 -> 31.5 mm
- net /ENA: track 17.2 -> 24.8 mm
- net /Pin_led_2: track 15.5 -> 21.7 mm
- net Net-(D4-Pad1): track 44.7 -> 50.3 mm
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
Commit message: actualización menor, 21/9/22
Parts:
- moved J1 66.0 mm to (93.3, 30.1), turned to 0 degrees
- moved J9 59.1 mm to (93.3, 34.9), turned to 0 degrees
- moved J5 40.3 mm to (53.1, 32.5), turned to 0 degrees
- moved C4 34.4 mm to (35.1, 65.1)
- moved D1 34.4 mm to (42.2, 65.0)
- moved U1 34.4 mm to (48.8, 70.0)
- moved R1 34.4 mm to (50.1, 63.7)
- moved C1 32.8 mm to (35.1, 71.8)
- moved J3 25.1 mm to (31.9, 56.5)
- moved J2 23.9 mm to (27.9, 56.5)
- moved G*** 18.9 mm to (40.9, 30.5), turned to 0 degrees
- moved J4 16.8 mm to (38.6, 50.1)
- moved U2 16.8 mm to (51.8, 55.2)
- moved C2 16.8 mm to (33.5, 39.7)
- moved C3 16.8 mm to (38.6, 40.0)
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Connections:
- J2 pad 2: /Pin_led_2 -> /Pin_led_2 y 3
- J3 pad 2: /Pin_led_3 -> /Pin_led_2 y 3
- U3 pad 10: /buzzer -> /IN_1_STEP
- U3 pad 12: unconnected-(U3-Pad12) -> /Pin_led_2 y 3
- U3 pad 24: unconnected-(U3-Pad24) -> /IN4
- U3 pad 25: unconnected-(U3-Pad25) -> /IN3
- U3 pad 26: unconnected-(U3-Pad26) -> /ENA
- U3 pad 27: /Pin_led_3 -> unconnected-(U3-Pad27)
- U3 pad 28: /Pin_led_2 -> unconnected-(U3-Pad28)
- U3 pad 29: /IN_4_STEP -> unconnected-(U3-Pad29)
- U3 pad 30: /IN_3_STEP -> /IN1
- U3 pad 31: /IN_2_STEP -> /IN2
- U3 pad 32: /IN_1_STEP -> /ENB
- U3 pad 4: /IN4 -> unconnected-(U3-Pad4)
- U3 pad 5: /IN3 -> unconnected-(U3-Pad5)
- U3 pad 6: /ENA -> /buzzer
- U3 pad 7: /IN1 -> /IN_4_STEP
- U3 pad 8: /IN2 -> /IN_3_STEP
- U3 pad 9: /ENB -> /IN_2_STEP
Routing:
- net VCC: track 215.9 -> 256.7 mm
- net /Pin_led_2 y 3: track 0.00 -> 34.5 mm
- net /Pin_led_2: track 21.7 -> 0.00 mm
- net /Pin_led_3: track 15.1 -> 0.00 mm
- net /IN2: track 31.5 -> 19.9 mm
- net /ENB: track 36.8 -> 26.1 mm
- net /IN1: track 26.1 -> 17.0 mm
- net /IN4: track 37.2 -> 28.3 mm
- net /IN3: track 31.9 -> 24.6 mm
- net +BATT: track 24.2 -> 17.6 mm
- net /buzzer: track 23.2 -> 17.2 mm
- net +5V: track 154.1 -> 157.8 mm, vias 0 -> 1
- net /pin_IR: track 7.84 -> 4.58 mm
- net /ENA: track 24.8 -> 21.7 mm
- net /tx0: track 12.1 -> 9.49 mm
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
Commit message: actualización 25/9/22
Parts:
- removed J3: led rgb, EESTN5:Pin_Header_3
- J1, J2, J9: footprint EESTN5:Pin_Header_3 -> Connector_JST:JST_EH_B3B-EH-A_1x03_P2.50mm_Vertical
- J4: footprint EESTN5:Pin_Strip_5 -> Connector_JST:JST_EH_B5B-EH-A_1x05_P2.50mm_Vertical
- moved J4 5.02 mm to (38.4, 55.2)
- moved J2 2.48 mm to (27.7, 58.9)
Routing:
- net +5V: track 157.8 -> 160.6 mm
- net /pin_IR: track 4.58 -> 7.15 mm
- net /tx0: track 9.49 -> 11.9 mm
- net /Pin_led_1: track 9.24 -> 11.5 mm

Commit message: actualizacion 26/10/22
Parts:
- removed J9: salida emisor, Connector_JST:JST_EH_B3B-EH-A_1x03_P2.50mm_Vertical
- added J3: motor izq, EESTN5:BORNERA2_AZUL, F.Cu at (99.9, 80.0)
- added R2: 470, EESTN5:RES0.3, F.Cu at (94.1, 32.4)
- added R3: 470, EESTN5:RES0.3, F.Cu at (48.1, 58.4)
- C2: value 100u -> 220uf
- C3: value 100n -> 100u; footprint Capacitor_THT:C_Rect_L4.6mm_W2.0mm_P2.50mm_MKS02_FKP02 -> Capacitor_THT:CP_Radial_D5.0mm_P2.00mm
- C4: value 220uf -> 100n; footprint Capacitor_THT:CP_Radial_D5.0mm_P2.00mm -> Capacitor_THT:C_Rect_L4.6mm_W2.0mm_P2.50mm_MKS02_FKP02
- J1: value led rgb -> buzzer; footprint Connector_JST:JST_EH_B3B-EH-A_1x03_P2.50mm_Vertical -> EESTN5:Pin_strip_2
- J2: value led rgb -> conector a stepper; footprint Connector_JST:JST_EH_B3B-EH-A_1x03_P2.50mm_Vertical -> Connector_JST:JST_EH_B5B-EH-A_1x05_P2.50mm_Vertical
- J4: value conector a stepper -> motor der; footprint Connector_JST:JST_EH_B5B-EH-A_1x05_P2.50mm_Vertical -> EESTN5:BORNERA2_AZUL
- J5: value buzzer -> bateria; footprint EESTN5:Pin_strip_2 -> EESTN5:BORNERA2_AZUL
- J6: value motor izq -> led rgb; footprint EESTN5:BORNERA2_AZUL -> Connector_JST:JST_EH_B3B-EH-A_1x03_P2.50mm_Vertical
- J7: value motor der -> led rgb; footprint EESTN5:BORNERA2_AZUL -> Connector_JST:JST_EH_B3B-EH-A_1x03_P2.50mm_Vertical
- J8: value bateria -> salida emisor; footprint EESTN5:BORNERA2_AZUL -> Connector_JST:JST_EH_B3B-EH-A_1x03_P2.50mm_Vertical
- moved J7 86.7 mm to (27.9, 58.9), turned to 90 degrees
- moved J4 77.5 mm to (111.8, 79.9), turned to 0 degrees
- moved J8 60.1 mm to (95.7, 39.5), turned to 180 degrees
- moved J6 52.4 mm to (95.4, 27.7)
- moved J5 50.0 mm to (39.6, 80.6)
- moved J1 40.4 mm to (53.0, 32.3)
- moved C5 38.9 mm to (91.4, 68.0)
- moved C4 32.4 mm to (47.0, 35.0), turned to 0 degrees
- moved C2 24.5 mm to (35.1, 64.2), turned to 180 degrees
- moved U4 22.2 mm to (114.2, 36.3), turned to -90 degrees
- moved C1 19.3 mm to (54.1, 75.3)
- moved U1 11.5 mm to (54.5, 80.0), turned to 180 degrees
- moved J2 11.5 mm to (38.5, 55.2)
- moved switch1 8.49 mm to (37.1, 71.7), turned to 90 degrees
- moved G*** 2.34 mm to (39.5, 28.6)
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Connections:
- C2 pad 1: VCC -> +5V
- C4 pad 1: +5V -> VCC
- J1 pad 1: +5V -> GND
- J1 pad 2: /Pin_led_1 -> /buzzer
- J2 pad 1: +5V -> Net-(J2-Pad1)
- J2 pad 2: /Pin_led_2 y 3 -> Net-(J2-Pad2)
- J2 pad 3: GND -> Net-(J2-Pad3)
- J4 pad 1: Net-(J4-Pad1) -> Net-(D6-Pad1)
- J4 pad 2: Net-(J4-Pad2) -> Net-(D8-Pad1)
- J5 pad 1: GND -> +BATT
- J5 pad 2: /buzzer -> GND
- J6 pad 1: Net-(D4-Pad1) -> +5V
- J6 pad 2: Net-(D2-Pad1) -> Net-(J6-Pad2)
- J7 pad 1: Net-(D6-Pad1) -> +5V
- J7 pad 2: Net-(D8-Pad1) -> Net-(J7-Pad2)
- J8 pad 1: +BATT -> /pin_IR
- J8 pad 2: GND -> /tx0
- U2 pad 13: Net-(J4-Pad4) -> Net-(J2-Pad4)
- U2 pad 14: Net-(J4-Pad3) -> Net-(J2-Pad3)
- U2 pad 15: Net-(J4-Pad2) -> Net-(J2-Pad2)
- U2 pad 16: Net-(J4-Pad1) -> Net-(J2-Pad1)
Routing:
- net Net-(C5-Pad2): track 81.7 -> 17.0 mm
- net VCC: track 256.8 -> 210.0 mm
- net /ENB: track 26.1 -> 67.6 mm
- net /IN2: track 19.9 -> 56.4 mm
- net /IN1: track 17.0 -> 48.0 mm
- net +5V: track 160.6 -> 188.1 mm, vias 1 -> 0
- net /Pin_led_2 y 3: track 34.8 -> 9.73 mm
- net Net-(J7-Pad2): track 0.00 -> 17.3 mm
- net Net-(D4-Pad1): track 50.2 -> 63.8 mm
- net +BATT: track 17.6 -> 8.99 mm
- net /Pin_led_1: track 11.5 -> 4.04 mm
- net /ENA: track 21.7 -> 29.1 mm
- net /pin_IR: track 7.15 -> 13.3 mm
- net Net-(J4-Pad1): track 5.73 -> 0.00 mm
- net Net-(J2-Pad1): track 0.00 -> 5.72 mm
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