File: kicad PCBs/car-complex/car-complex.kicad_sch (KiCad schematic)
At the start: 28 parts, among them J1 led rgb, J2 led rgb, J3 led rgb, J4 Conn_01x05_Male, J5 buzzer, J6 TB_1X2, J7 TB_1X2, J8 TB_1X2, J9 salida emisor, SW1 SW_SPDT, U1 LM78M05, U2 ULN2003A, U3 ESP32_DevKit_V1_DOIT, U4 L298(H)N

Commit message: actualización 19/09/2022
Parts:
- removed C1, C4: 220uf, EESTN5:CAP_ELEC_10X8mm, symbol Device:C_Polarized
- added C1: 10uf, Capacitor_THT:CP_Radial_D5.0mm_P2.00mm, symbol StepperDriver-rescue:CP_Small-Device
- added C4, C5: 220uf, Capacitor_THT:CP_Radial_D5.0mm_P2.00mm, symbol StepperDriver-rescue:CP_Small-Device
- D2, D3, D4, D5, D6, D7, D8, D9: value DIODE -> 1n4001
- J4: value Conn_01x05_Male -> conector a stepper
- J6: value TB_1X2 -> motor izq
- J7: value TB_1X2 -> motor der
- J8: value TB_1X2 -> bateria
- R1: value R -> 1k
- renumbered SW1 to switch1
Connections:
- net +5V: now also C4.1
- net ENA: now also U3.6 (IO32); no longer U3.8 (IO25)
- net ENB: now also U3.9 (IO26); no longer U3.11 (IO14)
- net GND: now also C1.2, C4.2
- net IN1: now also U3.7 (IO33); no longer U3.9 (IO26)
- net IN2: now also U3.8 (IO25); no longer U3.10 (IO27)
- net IN3: now also U3.5 (IO35); no longer U3.7 (IO33)
- net IN4: now also U3.4 (IO34); no longer U3.6 (IO32)
- net Pin_led_1: now also U3.36 (IO23); no longer U3.26 (IO4)
- net Pin_led_2: now also U3.28 (TX2); no longer U3.25 (IO2)
- net Pin_led_3: now also U3.27 (RX2); no longer U3.24 (IO15)
- net VCC: now also C1.1, C5.1
- net buzzer: now also U3.10 (IO27); no longer U3.12 (IO12)
- net at D3.1 (A), D5.1 (A), D7.1 (A)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: now also C5.2
Other:
- note added: "7.4v-8.4v"
- note added: "ESP32-pinout + buzzer"
- note removed: "ESP32"
- moved on the sheet: J5, J6, J7, U3

Commit message: actualización menor, 21/9/22
Connections:
- net ENA: now also U3.26 (IO4); no longer U3.6 (IO32)
- net ENB: now also U3.32 (IO21); no longer U3.9 (IO26)
- net IN1: now also U3.30 (IO18); no longer U3.7 (IO33)
- net IN2: now also U3.31 (IO19); no longer U3.8 (IO25)
- net IN3: now also U3.25 (IO2); no longer U3.5 (IO35)
- net IN4: now also U3.24 (IO15); no longer U3.4 (IO34)
- net IN_1_STEP: now also U3.10 (IO27); no longer U3.32 (IO21)
- net IN_2_STEP: now also U3.9 (IO26); no longer U3.31 (IO19)
- net IN_3_STEP: now also U3.8 (IO25); no longer U3.30 (IO18)
- net IN_4_STEP: now also U3.7 (IO33); no longer U3.29 (IO5)
- net buzzer: now also U3.6 (IO32); no longer U3.10 (IO27)
- net Pin_led_2 y 3: now reaches U3.12 (IO12)
- net Pin_led_2 y 3: now also J2.2 (P2), J3.2 (P2)
- net Pin_led_2: no longer names the net of U3.28 (TX2)
- net Pin_led_2: no longer J2.2 (P2)
- net Pin_led_3: no longer names the net of U3.27 (RX2)
- net Pin_led_3: no longer J3.2 (P2)
Other:
- moved on the sheet: J1, J2, J3

Commit message: actualización 25/9/22
Parts:
- removed J3: led rgb, EESTN5:Pin_Header_3, symbol EESTN5:CONN_01X03
- J1, J2, J9: footprint EESTN5:Pin_Header_3 -> Connector_JST:JST_EH_B3B-EH-A_1x03_P2.50mm_Vertical
- J4: footprint EESTN5:Pin_Strip_5 -> Connector_JST:JST_EH_B5B-EH-A_1x05_P2.50mm_Vertical
Changed lines of the file:
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@@
     (stroke (width 0) (type default) (color 0 0 0 0))
   )
-  (wire (pts (xy 252.73 265.43) (xy 255.27 265.43))
-    (stroke (width 0) (type default) (color 0 0 0 0))
-  )
   (wire (pts (xy 26.67 237.49) (xy 35.56 237.49))
     (stroke (width 0) (type default) (color 0 0 0 0))
@@
     (stroke (width 0) (type default) (color 0 0 0 0))
   )
-  (wire (pts (xy 252.73 262.89) (xy 255.27 262.89))
-    (stroke (width 0) (type default) (color 0 0 0 0))
-  )
   (wire (pts (xy 45.72 237.49) (xy 52.07 237.49))
     (stroke (width 0) (type default) (color 0 0 0 0))
@@
     (stroke (width 0) (type default) (color 0 0 0 0))
   )
-  (wire (pts (xy 252.73 267.97) (xy 255.27 267.97))
-    (stroke (width 0) (type default) (color 0 0 0 0))
-  )
   (polyline (pts (xy 16.51 281.94) (xy 16.51 201.93))
     (stroke (width 0) (type default) (color 0 0 0 0))
@@
     (effects (font (size 1.27 1.27)) (justify right bottom))
   )
-  (label "Pin_led_2 y 3" (at 252.73 265.43 180)
-    (effects (font (size 1.27 1.27)) (justify right bottom))
-  )
   (label "IN_1_STEP" (at 41.91 165.1 180)
     (effects (font (size 1.27 1.27)) (justify right bottom))
@@
       (effects (font (size 1.27 1.27)) (justify left))
     )
-    (property "Footprint" "EESTN5:Pin_Header_3" (id 2) (at 232.41 265.43 0)
+    (property "Footprint" "Connector_JST:JST_EH_B3B-EH-A_1x03_P2.50mm_Vertical" (id 2) (at 232.41 265.43 0)
       (effects (font (size 1.27 1.27)) hide)
     )
@@
     (pin "2")
   )
-  (symbol (lib_id "power:+5V") (at 252.73 262.89 0) (unit 1)
-    (in_bom yes) (on_board yes) (fields_autoplaced)
-    (property "Reference" "#PWR0110" (id 0) (at 252.73 266.7 0)
-      (effects (font (size 1.27 1.27)) hide)
-    )
-    (property "Value" "+5V" (id 1) (at 252.73 257.81 0))
-    (property "Footprint" "" (id 2) (at 252.73 262.89 0)
-      (effects (font (size 1.27 1.27)) hide)
-    )
-    (property "Datasheet" "" (id 3) (at 252.73 262.89 0)
-      (effects (font (size 1.27 1.27)) hide)
-    )
-    (pin "1")
-  )
   (symbol (lib_id "EESTN5:DIODE") (at 120.65 264.16 90) (unit 1)
     (in_bom yes) (on_board yes)
@@
       (effects (font (size 1.27 1.27)) (justify right))
     )
-    (property "Footprint" "EESTN5:Pin_Strip_5" (id 2) (at 115.57 167.64 0)
+    (property "Footprint" "Connector_JST:JST_EH_B5B-EH-A_1x05_P2.50mm_Vertical" (id 2) (at 115.57 167.64 0)
       (effects (font (size 1.27 1.27)) hide)
     )
@@
       (effects (font (size 1.27 1.27)) (justify left))
     )
-    (property "Footprint" "EESTN5:Pin_Header_3" (id 2) (at 204.47 265.43 0)
+    (property "Footprint" "Connector_JST:JST_EH_B3B-EH-A_1x03_P2.50mm_Vertical" (id 2) (at 204.47 265.43 0)
       (effects (font (size 1.27 1.27)) hide)
     )
@@
       (effects (font (size 1.27 1.27)) (justify left))
     )
-    (property "Footprint" "EESTN5:Pin_Header_3" (id 2) (at 267.97 229.87 0)
+    (property "Footprint" "Connector_JST:JST_EH_B3B-EH-A_1x03_P2.50mm_Vertical" (id 2) (at 267.97 229.87 0)
       (effects (font (size 1.27 1.27)) hide)
     )
@@
     (pin "3")
   )
-  (symbol (lib_id "EESTN5:CONN_01X03") (at 260.35 265.43 0) (unit 1)
-    (in_bom yes) (on_board yes)
-    (property "Reference" "J3" (id 0) (at 262.89 264.1599 0)
-      (effects (font (size 1.27 1.27)) (justify left))
-    )
-    (property "Value" "led rgb" (id 1) (at 256.54 270.51 0)
-      (effects (font (size 1.27 1.27)) (justify left))
-    )
-    (property "Footprint" "EESTN5:Pin_Header_3" (id 2) (at 260.35 265.43 0)
-      (effects (font (size 1.27 1.27)) hide)
-    )
-    (property "Datasheet" "" (id 3) (at 260.35 265.43 0)
-      (effects (font (size 1.27 1.27)) hide)
-    )
-    (pin "1")
-    (pin "2")
-    (pin "3")
-  )
-  (symbol (lib_id "power:GND") (at 252.73 267.97 0) (unit 1)
-    (in_bom yes) (on_board yes) (fields_autoplaced)
-    (property "Reference" "#PWR0106" (id 0) (at 252.73 274.32 0)
-      (effects (font (size 1.27 1.27)) hide)
-    )
-    (property "Value" "GND" (id 1) (at 252.73 273.05 0))
-    (property "Footprint" "" (id 2) (at 252.73 267.97 0)
-      (effects (font (size 1.27 1.27)) hide)
-    )
-    (property "Datasheet" "" (id 3) (at 252.73 267.97 0)
-      (effects (font (size 1.27 1.27)) hide)
-    )
-    (pin "1")
-  )
   (symbol (lib_id "power:GND") (at 50.8 97.79 0) (unit 1)
     (in_bom yes) (on_board yes) (fields_autoplaced)
@@
       (reference "#PWR0105") (unit 1) (value "GND") (footprint "")
     )
-    (path "/f0ff0792-4d97-4881-9b9c-759645b25c42"
-      (reference "#PWR0106") (unit 1) (value "GND") (footprint "")
-    )
     (path "/0247a021-bc0f-417c-b3cd-69e691982415"
       (reference "#PWR0107") (unit 1) (value "GND") (footprint "")
@@
       (reference "#PWR0109") (unit 1) (value "GND") (footprint "")
     )
-    (path "/87787b7b-0950-4e3b-8130-4503b072059b"
-      (reference "#PWR0110") (unit 1) (value "+5V") (footprint "")
-    )
     (path "/5f126e9b-7563-484c-83aa-2450540d588a"
       (reference "#PWR0111") (unit 1) (value "GND") (footprint "")
@@
     )
     (path "/dae881eb-5d09-40cc-889c-e19fe13bfa5f"
-      (reference "J1") (unit 1) (value "led rgb") (footprint "EESTN5:Pin_Header_3")
+      (reference "J1") (unit 1) (value "led rgb") (footprint "Connector_JST:JST_EH_B3B-EH-A_1x03_P2.50mm_Vertical")
     )
     (path "/0ff704c6-a2dd-4809-b2af-62f6c5cbf333"
-      (reference "J2") (unit 1) (value "led rgb") (footprint "EESTN5:Pin_Header_3")
-    )
-    (path "/ed7c54c8-eb1f-4548-b828-59ecb89c3d82"
-      (reference "J3") (unit 1) (value "led rgb") (footprint "EESTN5:Pin_Header_3")
+      (reference "J2") (unit 1) (value "led rgb") (footprint "Connector_JST:JST_EH_B3B-EH-A_1x03_P2.50mm_Vertical")
     )
     (path "/bffcb526-91c6-4305-a053-a1ecc5566243"
-      (reference "J4") (unit 1) (value "conector a stepper") (footprint "EESTN5:Pin_Strip_5")
+      (reference "J4") (unit 1) (value "conector a stepper") (footprint "Connector_JST:JST_EH_B5B-EH-A_1x05_P2.50mm_Vertical")
     )
     (path "/305ea261-fce3-4c69-be1a-aa4df964d8cb"
@@
     )
     (path "/ed2384fc-6457-4bc7-92ac-dc092fe243b4"
-      (reference "J9") (unit 1) (value "salida emisor") (footprint "EESTN5:Pin_Header_3")
+      (reference "J9") (unit 1) (value "salida emisor") (footprint "Connector_JST:JST_EH_B3B-EH-A_1x03_P2.50mm_Vertical")
     )
     (path "/5674be13-8670-4f78-839f-ca23d53d1871"

Commit message: actualizacion 26/10/22
Parts:
- added R2, R3: 470, EESTN5:RES0.3, symbol EESTN5:R
- renumbered C4 to C2, C2 to C3, C3 to C4, J5 to J1, J4 to J2, J6 to J3, J7 to J4, J8 to J5, J1 to J6, J2 to J7, J9 to J8
Connections:
- net Pin_led_1: now also R2.1; no longer J6.2 (P2)
- net Pin_led_2 y 3: now also R3.1; no longer J7.2 (P2)
- new net: J7.2 (P2), R3.2
- new net: J6.2 (P2), R2.2
Other:
- moved on the sheet: J6, J7
